File: Schematics/Joystick Controller Board/Joystick Controller.brd (EAGLE design)
At the start: 41.6 x 80 mm, 7 parts, among them U1 TEENSY2-ARDUINO, U2 JOYSTICKPTH

Commit message: Schematics updated External Controller board schematic created
Other:
- board text added: "Joystick Controller Board V1"
Changed lines of the file:
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@@
 <wire x1="41.58" y1="80" x2="0" y2="80" width="0" layer="20"/>
 <wire x1="0" y1="80" x2="0" y2="0" width="0" layer="20"/>
+<text x="11.43" y="73.66" size="1.778" layer="25">Joystick Controller
+Board V1</text>
 </plain>
 <attributes>
@@
 </board>
 </drawing>
+<compatibility>
+<note version="6.3" minversion="6.2.2" severity="warning">
+Since Version 6.2.2 text objects can contain more than one line,
+which will not be processed correctly with this version.
+</note>
+</compatibility>
 </eagle>
