File: Schematics/Power Board/Power Board.brd (EAGLE design)
At the start: 25.1 x 52.1 mm, 7 parts

Commit message: Schematics updated External Controller board schematic created
Other:
- board text added: "Power Board V1"
Changed lines of the file:
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@@
 <text x="22.86" y="20.32" size="1.778" layer="25">+</text>
 <text x="24.13" y="29.21" size="1.778" layer="25" rot="R90">-</text>
+<text x="21.59" y="1.27" size="1.778" layer="25" rot="R90">Power Board V1</text>
 </plain>
 <attributes>
